Commit message: Benchmark: Success fixed body on some DOFs

File: simulation/models/carwheel/urdf/carwheel_constraint.urdf (robot description, URDF)
Before this commit: robot carwheel, 5 links, 4 joints
Links:
- added link virtual_body, mass 0.00001
- added link virtual_pz_link, mass 0.00001
- added link world
Joints:
- added joint virtual_fixed_joint: type fixed, parent virtual_body, child real_body
- added joint virtual_px_joint: type prismatic, parent virtual_pz_link, child virtual_body, origin xyz=0 0 0 rpy=0 0 0, axis 1 0 0, limit lower=-1000.0 upper=1000.0 effort=1000.0 velocity=1000.0
- added joint virtual_pz_joint: type prismatic, parent world, child virtual_pz_link, origin xyz=0 0 0 rpy=0 0 0, axis 0 0 1, limit lower=-10.0 upper=10.0 effort=100.0 velocity=1000.0
