Commit message: Benchmark: Success add velocity based controller in gazebo

File: simulation/models/carwheel/urdf/carwheel.urdf (robot description, URDF)
Before this commit: robot carwheel, 5 links, 4 joints
Joints:
- joint Joint_FL: limit lower=-1000000 upper=1000000 effort=30 velocity=20 -> lower=-1000000 upper=1000000 effort=100 velocity=1000
- joint Joint_FR: limit lower=-1000000 upper=1000000 effort=30 velocity=20 -> lower=-1000000 upper=1000000 effort=100 velocity=1000
- joint Joint_HL: limit lower=-1000000 upper=1000000 effort=30 velocity=20 -> lower=-1000000 upper=1000000 effort=100 velocity=1000
- joint Joint_HR: limit lower=-1000000 upper=1000000 effort=30 velocity=20 -> lower=-1000000 upper=1000000 effort=100 velocity=1000

Commit message: Benchmark: Success add torque based controller in gazebo

File: simulation/models/carwheel/urdf/carwheel.urdf (robot description, URDF)
Before this commit: robot carwheel, 5 links, 4 joints
Joints:
- joint Joint_FL: limit lower=-1000000 upper=1000000 effort=100 velocity=1000 -> lower=-1000000 upper=1000000 effort=50 velocity=200
- joint Joint_FR: limit lower=-1000000 upper=1000000 effort=100 velocity=1000 -> lower=-1000000 upper=1000000 effort=50 velocity=200
- joint Joint_HL: limit lower=-1000000 upper=1000000 effort=100 velocity=1000 -> lower=-1000000 upper=1000000 effort=50 velocity=200
- joint Joint_HR: limit lower=-1000000 upper=1000000 effort=100 velocity=1000 -> lower=-1000000 upper=1000000 effort=50 velocity=200
